File: one_dollar_boad.sch (EAGLE design)
At the start: 37 parts, among them IC1 ATTINY85, X1 USBPCB

Commit message: `
- Adicionado slot para LD1117
- Adicionado Silk
- Cantos chanfrados
- Retirado GND dos componentes de expansão para que o usuário possa usar os expansores que achar melhor.
Parts:
- added EX1: (no value), con-amp:MTA04-100
- added J9: (no value), con-amp:MTA03-100
- J3: device con-amp:MTA04-100 -> con-amp:MTA03-100
- renumbered 24C256 to EX2, L293D to EX3
Connections:
- new net N$46: J4.4, U$8.GND
- new net N$47: EX2.GND, J5.1
- new net N$48: EX3.GND2, J2.4
- new net N$49: EX3.GND4, J1.5
- new net N$50: EX3.GND3, J1.4
- new net N$51: EX3.GND1, J2.5
- new net N$52: J3.1, J9.3
- new net N$53: J3.2, J9.2
- new net N$54: J3.3, J9.1
- net GND: no longer EX2.GND, EX3.GND1, EX3.GND2, EX3.GND3, EX3.GND4, J1.4, J1.5, J2.4, J2.5, J4.4, U$8.GND
- net N$32: now also EX1.1; no longer J3.1
- net N$33: now also EX1.2; no longer J3.2
- net N$34: now also EX1.3; no longer J3.3
- net N$35: now also EX1.4; no longer J3.4
Other:
- note removed: "Created by Erik Kettenbugr, Digistump LLC - digistump.com 2012"
- note removed: "Digispark name. logo and Digistump name, logo Copyright 2013 Digistump LLC All Rights Reserved"
- note removed: "For full details and license information please see http://digistump.com/wiki/digispark/policy"
- note removed: "The Digispark and Digistump names and logos (or derivatives thereof) may not be used as part of the name of a product, company, or domain name without express written permission."
- note removed: "The Digispark design (schematic, layout, concept) is licensed under the Creative Commons Attribution-ShareAlike 3.0 Unported License: http://creativecommons.org/licenses/by-sa/3.0/"
