File: one_dollar_boad_beta4.brd (EAGLE design)
At the start: 85.6 x 54 mm, 39 parts, among them IC1 ATTINY85, X1 USBPCB

Commit message: Modificação feita por Marcelo Cuin
Parts:
- CONNECTORBAR1: value FAMALEBAR01X08 -> .
- moved J10 0.80 mm to (79.2, 18.9)
- moved J9 0.40 mm to (79.2, 23.5)
Other:
- board text added: "1"
- board text added: "2"
- board text added: "3"
- board text added: "4"
- board text added: "5"
- board text added: "5v"
- board text added: "6"
- board text added: "7"
- board text added: "8"
- board text added: "gnd"
- board text added: "p0"
- board text added: "p1"
- board text added: "p2"
- board text added: "p3"
- board text added: "p4"
- board text added: "p5"
Changed lines of the file:
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@@
 <?xml version="1.0" encoding="utf-8"?>
 <!DOCTYPE eagle SYSTEM "eagle.dtd">
-<eagle version="7.5.0">
+<eagle version="7.2.0">
 <drawing>
 <settings>
@@
 <layer number="23" name="tOrigins" color="15" fill="1" visible="yes" active="yes"/>
 <layer number="24" name="bOrigins" color="15" fill="1" visible="no" active="yes"/>
-<layer number="25" name="tNames" color="7" fill="1" visible="yes" active="yes"/>
-<layer number="26" name="bNames" color="7" fill="1" visible="yes" active="yes"/>
-<layer number="27" name="tValues" color="7" fill="1" visible="no" active="yes"/>
+<layer number="25" name="tNames" color="7" fill="1" visible="no" active="yes"/>
+<layer number="26" name="bNames" color="7" fill="1" visible="no" active="yes"/>
+<layer number="27" name="tValues" color="7" fill="1" visible="yes" active="yes"/>
 <layer number="28" name="bValues" color="7" fill="1" visible="no" active="yes"/>
 <layer number="29" name="tStop" color="7" fill="3" visible="no" active="yes"/>
@@
 <wire x1="83.3" y1="0" x2="85.6" y2="2.3" width="0.254" layer="21" curve="90"/>
 <wire x1="14.5" y1="0" x2="12" y2="2.5" width="0.254" layer="21" curve="-90"/>
+<text x="19.2" y="51.1" size="1.016" layer="27">5v</text>
+<wire x1="19.7" y1="44.1" x2="19.7" y2="50.7" width="0.15" layer="27"/>
+<wire x1="22.3" y1="44.1" x2="22.3" y2="50.7" width="0.15" layer="27"/>
+<wire x1="24.8" y1="44.1" x2="24.8" y2="50.7" width="0.15" layer="27"/>
+<wire x1="27.3" y1="44" x2="27.3" y2="50.6" width="0.15" layer="27"/>
+<wire x1="29.9" y1="44" x2="29.9" y2="50.6" width="0.15" layer="27"/>
+<wire x1="32.4" y1="44" x2="32.4" y2="50.6" width="0.15" layer="27"/>
+<wire x1="35" y1="44" x2="35" y2="50.6" width="0.15" layer="27"/>
+<wire x1="37.5" y1="44" x2="37.5" y2="50.6" width="0.15" layer="27"/>
+<text x="21.1" y="51.1" size="1.016" layer="27">gnd</text>
+<text x="24.1" y="51.1" size="1.016" layer="27">p0</text>
+<text x="26.6" y="51" size="1.016" layer="27">p1</text>
+<text x="29.1" y="51" size="1.016" layer="27">p2</text>
+<text x="31.6" y="50.9" size="1.016" layer="27">p3</text>
+<text x="34.2" y="50.9" size="1.016" layer="27">p4</text>
+<text x="36.7" y="50.9" size="1.016" layer="27">p5</text>
+<text x="71.1" y="0.3" size="0.8128" layer="27">1</text>
+<text x="73.6" y="0.3" size="0.8128" layer="27">2</text>
+<text x="76" y="0.3" size="0.8128" layer="27">3</text>
+<text x="78.6" y="0.3" size="0.8128" layer="27">4</text>
+<text x="70.4" y="5.2" size="0.8128" layer="27">5</text>
+<text x="73" y="5.2" size="0.8128" layer="27">6</text>
+<text x="75.5" y="5.2" size="0.8128" layer="27">7</text>
+<text x="78.2" y="5.4" size="0.8128" layer="27">8</text>
+<text x="71.1" y="16.1" size="0.8128" layer="27">1</text>
+<text x="73.6" y="16.1" size="0.8128" layer="27">2</text>
+<text x="76.2" y="16.1" size="0.8128" layer="27">3</text>
+<text x="78.7" y="16.1" size="0.8128" layer="27">4</text>
+<text x="71" y="10.8" size="0.8128" layer="27">5</text>
+<text x="73.6" y="10.8" size="0.8128" layer="27">6</text>
+<text x="76.2" y="10.8" size="0.8128" layer="27">7</text>
+<text x="78.7" y="10.8" size="0.8128" layer="27">8</text>
 </plain>
 <attributes>
@@
 <element name="J7" library="con-amp" package="10X02MTA" value="" x="70.7898" y="21.1074"/>
 <element name="J8" library="con-amp" package="10X02MTA" value="" x="70.6374" y="51.0794" rot="R180"/>
-<element name="CONNECTORBAR1" library="femeabarra01x08" package="FEMEABARRA01X08" value="FAMALEBAR01X08" x="19.685" y="42.2274"/>
+<element name="CONNECTORBAR1" library="femeabarra01x08" package="FEMEABARRA01X08" value="." x="19.685" y="42.2274"/>
 <element name="U$9" library="arduinopinagem" package="ARDUINOPINAGEM" value="ARDUINOPINAGEM" x="31.0134" y="2.7686"/>
 <element name="ICSP1" library="ICSP" package="ICSP" value="ICSP" x="37.2" y="37"/>
@@
 <element name="ICSP6" library="ICSP" package="ICSP" value="ICSP" x="30" y="31.8"/>
 <element name="R6" library="SparkFun" package="0402-RES" value="" x="33.8" y="17" rot="R270"/>
-<element name="J9" library="con-amp" package="10X03MTA" value="" x="79.2" y="23.9" rot="R180"/>
-<element name="J10" library="con-amp" package="10X03MTA" value="" x="79.2" y="19.7"/>
+<element name="J9" library="con-amp" package="10X03MTA" value="" x="79.2" y="23.5" rot="R180"/>
+<element name="J10" library="con-amp" package="10X03MTA" value="" x="79.2" y="18.9"/>
 </elements>
 <signals>
@@
 <contactref element="J10" pad="3"/>
 <contactref element="J9" pad="1"/>
-<wire x1="76.66" y1="19.7" x2="76.66" y2="23.9" width="0.254" layer="1"/>
+<wire x1="76.66" y1="18.9" x2="76.66" y2="23.5" width="0.254" layer="1"/>
 </signal>
 <signal name="N$41">
 <contactref element="J10" pad="2"/>
 <contactref element="J9" pad="2"/>
-<wire x1="79.2" y1="19.7" x2="79.2" y2="23.9" width="0.254" layer="1"/>
+<wire x1="79.2" y1="18.9" x2="79.2" y2="23.5" width="0.254" layer="1"/>
 </signal>
 <signal name="N$48">
 <contactref element="J10" pad="1"/>
 <contactref element="J9" pad="3"/>
-<wire x1="81.74" y1="19.7" x2="81.74" y2="23.9" width="0.254" layer="1"/>
+<wire x1="81.74" y1="18.9" x2="81.74" y2="23.5" width="0.254" layer="1"/>
 </signal>
 </signals>
